Commit message: cleaning up before updating gitignore

File: panda_starter_code/panda_arm.urdf (robot description, URDF)
Before this commit: robot panda, 8 links, 7 joints
Links:
- link link7: geometry collision sphere radius=0.03; visual mesh filename=../../../Model/meshes/EE_end.obj

Commit message: EE .obj did not work, revert back

File: panda_starter_code/panda_arm.urdf (robot description, URDF)
Before this commit: robot panda, 8 links, 7 joints
Links:
- link link7: geometry collision sphere radius=0.03; visual mesh filename=../../../Model/meshes/visual/link7.obj

Commit message: added crokiboard to world rendering as part of link0 visual

File: panda_starter_code/panda_arm.urdf (robot description, URDF)
Before this commit: robot panda, 8 links, 7 joints
Links:
- link link0: geometry visual mesh filename=../../../Model/meshes/crokiboard.obj; visual mesh filename=../../../Model/meshes/visual/link0.obj

Commit message: Added end effector to robot urdf

File: panda_starter_code/panda_arm.urdf (robot description, URDF)
Before this commit: robot panda, 8 links, 7 joints
Links:
- link link7: geometry visual mesh filename=../../../Model/meshes/Endeffector.obj scale=0.0013 0.0013 0.0013

Commit message: changed robot end effector in urdf

File: panda_starter_code/panda_arm.urdf (robot description, URDF)
Before this commit: robot panda, 8 links, 7 joints
Links:
- link link7: geometry visual mesh filename=../../../Model/meshes/endeffector_short.obj scale=0.0013 0.0013 0.0013

Commit message: added new end effector to simulation

File: panda_starter_code/panda_arm.urdf (robot description, URDF)
Before this commit: robot panda, 8 links, 7 joints
Links:
- link link7: geometry visual mesh filename=../../../Model/meshes/Assembly_sideEE.obj scale=0.0013 0.0013 0.0013

Commit message: EE orientation tests

File: panda_starter_code/panda_arm.urdf (robot description, URDF)
Before this commit: robot panda, 8 links, 7 joints
Links:
- link link7: geometry visual mesh filename=../../../Model/meshes/Assembly_sideEE.obj scale=0.001 0.001 0.001

Commit message: added new EE to sim

File: panda_starter_code/panda_arm.urdf (robot description, URDF)
Before this commit: robot panda, 8 links, 7 joints
Links:
- link link7: geometry visual mesh filename=../../../Model/meshes/newEE.obj scale=0.001 0.001 0.001
